Commit message: meio do caminho lesgo

File: urdf/model_backup.urdf (robot description, URDF)
Before this commit: robot quadrupedal_robot, 22 links, 21 joints
Links:
- link base_link: geometry collision box size=4 1.5 .5; visual box size=4 1.5 .5
- link left_back_calf: geometry collision cylinder length=2 radius=.1; visual cylinder length=2 radius=.1
- link left_back_elbow_ball: geometry collision sphere radius=.1; visual sphere radius=.1
- link left_back_foot: geometry collision sphere radius=.1; visual sphere radius=.1
- link left_back_leg: geometry collision cylinder length=2 radius=.1; visual cylinder length=2 radius=.1
- link left_back_shoulder: geometry collision cylinder length=.05 radius=.1; visual cylinder length=.05 radius=.1
- link left_front_calf: geometry collision cylinder length=2 radius=.1; visual cylinder length=2 radius=.1
- link left_front_elbow_ball: geometry collision sphere radius=.1; visual sphere radius=.1
- link left_front_foot: geometry collision sphere radius=.1; visual sphere radius=.1
- link left_front_leg: geometry collision cylinder length=2 radius=.1; visual cylinder length=2 radius=.1
- link left_front_shoulder: geometry collision cylinder length=.05 radius=.1; visual cylinder length=.05 radius=.1
- link right_back_calf: geometry collision cylinder length=2 radius=.1; visual cylinder length=2 radius=.1
- link right_back_elbow_ball: geometry collision sphere radius=.1; visual sphere radius=.1
- link right_back_foot: geometry collision sphere radius=.1; visual sphere radius=.1
- link right_back_leg: geometry collision cylinder length=2 radius=.1; visual cylinder length=2 radius=.1
- link right_back_shoulder: geometry collision cylinder length=.05 radius=.1; visual cylinder length=.05 radius=.1
- link right_front_calf: geometry collision cylinder length=2 radius=.1; visual cylinder length=2 radius=.1
- link right_front_elbow_ball: geometry collision sphere radius=.1; visual sphere radius=.1
- link right_front_foot: geometry collision sphere radius=.1; visual sphere radius=.1
- link right_front_leg: geometry collision cylinder length=2 radius=.1; visual cylinder length=2 radius=.1
- link right_front_shoulder: geometry collision cylinder length=.05 radius=.1; visual cylinder length=.05 radius=.1
Joints:
- joint left_back_calf_elbow_hinge: axis 0 0 1 -> 0 1 0; limit lower=-1.57 upper=1.57 effort=1 velocity=1 -> lower=-.79 upper=.79 effort=1000 velocity=1; origin xyz=0 0 0 rpy=0 0 0 -> xyz=0 0 -.2 rpy=0 0 0
- joint left_back_foot_hinge: origin xyz=0.35 0 0 rpy=0 0 0 -> xyz=0 0 -2 rpy=0 0 0
- joint left_back_leg_elbow_hinge: axis 0 0 1 -> 0 1 0; limit lower=-1.57 upper=1.57 effort=1 velocity=1 -> lower=-.79 upper=.79 effort=1000 velocity=1; origin xyz=0.4 0 0 rpy=1.57 0 0 -> xyz=0 0 -1.9 rpy=0 0 0
- joint left_back_leg_shoulder_hinge: axis 0 0 1 -> 1 0 0; limit lower=-1.57 upper=1.57 effort=1 velocity=1 -> lower=-.52 upper=1.57 effort=1000 velocity=1; origin xyz=0 0 0.1 rpy=-1.57 0 -1.57 -> xyz=0 .125 0 rpy=0 0 0
- joint left_back_leg_shoulder_rotate: axis 0 0 1 -> 0 1 0; limit lower=-1.57 upper=1.57 effort=1 velocity=1 -> lower=-1.57 upper=1.57 effort=1000 velocity=1; origin xyz=-0.5 0.2 0 rpy=-1.57 3.14 0 -> xyz=-1.5 .75 0 rpy=0 0 0
- joint left_front_calf_elbow_hinge: axis 0 0 1 -> 0 1 0; limit lower=-1.57 upper=1.57 effort=1 velocity=1 -> lower=-.79 upper=.79 effort=1000 velocity=1; origin xyz=0 0 0 rpy=0 0 0 -> xyz=0 0 -.2 rpy=0 0 0
- joint left_front_foot_hinge: origin xyz=0.35 0 0 rpy=0 0 0 -> xyz=0 0 -2 rpy=0 0 0
- joint left_front_leg_elbow_hinge: axis 0 0 1 -> 0 1 0; limit lower=-1.57 upper=1.57 effort=1 velocity=1 -> lower=-.79 upper=.79 effort=1000 velocity=1; origin xyz=0.4 0 0 rpy=1.57 0 0 -> xyz=0 0 -1.9 rpy=0 0 0
- joint left_front_leg_shoulder_hinge: axis 0 0 1 -> 1 0 0; limit lower=-1.57 upper=1.57 effort=1 velocity=1 -> lower=-.52 upper=1.57 effort=1000 velocity=1; origin xyz=0 0 0.1 rpy=-1.57 0 -1.57 -> xyz=0 .125 0 rpy=0 0 0
- joint left_front_leg_shoulder_rotate: axis 0 0 1 -> 0 1 0; limit lower=-1.57 upper=1.57 effort=1 velocity=1 -> lower=-1.57 upper=1.57 effort=1000 velocity=1; origin xyz=0.5 0.2 0 rpy=-1.57 3.14 0 -> xyz=1.5 .75 0 rpy=0 0 0
- joint right_back_calf_elbow_hinge: axis 0 0 1 -> 0 1 0; limit lower=-1.57 upper=1.57 effort=1 velocity=1 -> lower=-.79 upper=.79 effort=1000 velocity=1; origin xyz=0 0 0 rpy=0 0 0 -> xyz=0 0 -.2 rpy=0 0 0
- joint right_back_foot_hinge: origin xyz=0.35 0 0 rpy=0 0 0 -> xyz=0 0 -2 rpy=0 0 0
- joint right_back_leg_elbow_hinge: axis 0 0 1 -> 0 1 0; limit lower=-1.57 upper=1.57 effort=1 velocity=1 -> lower=-.79 upper=.79 effort=1000 velocity=1; origin xyz=0.4 0 0 rpy=1.57 0 0 -> xyz=0 0 -1.9 rpy=0 0 0
- joint right_back_leg_shoulder_hinge: axis 0 0 1 -> 1 0 0; limit lower=-1.57 upper=1.57 effort=1 velocity=1 -> lower=-.52 upper=1.57 effort=1000 velocity=1; origin xyz=0 0 0.1 rpy=-1.57 0 -1.57 -> xyz=0 -.125 0 rpy=0 0 0
- joint right_back_leg_shoulder_rotate: axis 0 0 1 -> 0 1 0; limit lower=-1.57 upper=1.57 effort=1 velocity=1 -> lower=-1.57 upper=1.57 effort=1000 velocity=1; origin xyz=-0.5 -0.2 0 rpy=1.57 0 0 -> xyz=-1.5 -.75 0 rpy=0 0 0
- joint right_front_calf_elbow_hinge: axis 0 0 1 -> 0 1 0; limit lower=-1.57 upper=1.57 effort=1 velocity=1 -> lower=-.79 upper=.79 effort=1000 velocity=1; origin xyz=0 0 0 rpy=0 0 0 -> xyz=0 0 -.2 rpy=0 0 0
- joint right_front_foot_hinge: origin xyz=0.35 0 0 rpy=0 0 0 -> xyz=0 0 -2 rpy=0 0 0
- joint right_front_leg_elbow_hinge: axis 0 0 1 -> 0 1 0; limit lower=-1.57 upper=1.57 effort=1 velocity=1 -> lower=-.79 upper=.79 effort=1000 velocity=1; origin xyz=0.4 0 0 rpy=1.57 0 0 -> xyz=0 0 -1.9 rpy=0 0 0
- joint right_front_leg_shoulder_hinge: axis 0 0 1 -> 1 0 0; limit lower=-1.57 upper=1.57 effort=1 velocity=1 -> lower=-.52 upper=1.57 effort=1000 velocity=1; origin xyz=0 0 0.1 rpy=-1.57 0 -1.57 -> xyz=0 -.125 0 rpy=0 0 0
- joint right_front_leg_shoulder_rotate: axis 0 0 1 -> 0 1 0; limit lower=-1.57 upper=1.57 effort=1 velocity=1 -> lower=-1.57 upper=1.57 effort=1000 velocity=1; origin xyz=0.5 -0.2 0 rpy=1.57 0 0 -> xyz=1.5 -.75 0 rpy=0 0 0
