Commit message: commit 30/11

File: urdf/model2.urdf (robot description, URDF)
Before this commit: robot quadrupedal_robot, 22 links, 21 joints
Links:
- removed link left_back_elbow_ball
- removed link left_front_elbow_ball
- removed link right_back_elbow_ball
- removed link right_front_elbow_ball
- link base_link: geometry collision box size=1 0.4 .2; visual box size=1 0.4 .2
- link left_back_calf: geometry collision cylinder length=0.35 radius=.05; visual cylinder length=0.35 radius=.05
- link left_back_foot: geometry collision sphere radius=.05; visual sphere radius=.05
- link left_back_leg: geometry collision cylinder length=0.4 radius=.05; visual cylinder length=0.4 radius=.05
- link left_back_shoulder: geometry collision cylinder length=.1 radius=.05; visual cylinder length=.1 radius=.05
- link left_front_calf: geometry collision cylinder length=0.35 radius=.05; visual cylinder length=0.35 radius=.05
- link left_front_foot: geometry collision sphere radius=.05; visual sphere radius=.05
- link left_front_leg: geometry collision cylinder length=0.4 radius=.05; visual cylinder length=0.4 radius=.05
- link left_front_shoulder: geometry collision cylinder length=.1 radius=.05; visual cylinder length=.1 radius=.05
- link right_back_calf: geometry collision cylinder length=0.35 radius=.05; visual cylinder length=0.35 radius=.05
- link right_back_foot: geometry collision sphere radius=.05; visual sphere radius=.05
- link right_back_leg: geometry collision cylinder length=0.4 radius=.05; visual cylinder length=0.4 radius=.05
- link right_back_shoulder: geometry collision cylinder length=.1 radius=.05; visual cylinder length=.1 radius=.05
- link right_front_calf: geometry collision cylinder length=0.35 radius=.05; visual cylinder length=0.35 radius=.05
- link right_front_foot: geometry collision sphere radius=.05; visual sphere radius=.05
- link right_front_leg: geometry collision cylinder length=0.4 radius=.05; visual cylinder length=0.4 radius=.05
- link right_front_shoulder: geometry collision cylinder length=.1 radius=.05; visual cylinder length=.1 radius=.05
Joints:
- removed joint left_back_calf_elbow_hinge
- removed joint left_front_calf_elbow_hinge
- removed joint right_back_calf_elbow_hinge
- removed joint right_front_calf_elbow_hinge
- joint left_back_foot_hinge: origin xyz=0 0 -2 rpy=0 0 0 -> xyz=0.35 0 0 rpy=0 0 0
- joint left_back_leg_elbow_hinge: axis 0 1 0 -> 0 0 1; child left_back_elbow_ball -> left_back_calf; limit lower=-.79 upper=.79 effort=1000 velocity=1 -> lower=-1.57 upper=1.57 effort=100 velocity=1; origin xyz=0 0 -1.9 rpy=0 0 0 -> xyz=0.4 0 0 rpy=0 0 0
- joint left_back_leg_shoulder_hinge: axis 1 0 0 -> 0 0 1; child left_back_leg -> left_back_shoulder; limit lower=-.52 upper=1.57 effort=1000 velocity=1 -> lower=-1.57 upper=1.57 effort=100 velocity=1; origin xyz=0 .125 0 rpy=0 0 0 -> xyz=-0.5 .2 0 rpy=1.57 0 -1.57; parent left_back_shoulder -> base_link
- joint left_back_leg_shoulder_rotate: axis 0 1 0 -> 0 0 1; child left_back_shoulder -> left_back_leg; limit lower=-1.57 upper=1.57 effort=1000 velocity=1 -> lower=-1.57 upper=1.57 effort=100 velocity=1; origin xyz=-1.5 .75 0 rpy=0 0 0 -> xyz=-.1 0 0 rpy=1.57 0 -1.57; parent base_link -> left_back_shoulder
- joint left_front_foot_hinge: origin xyz=0 0 -2 rpy=0 0 0 -> xyz=0.35 0 0 rpy=0 0 0
- joint left_front_leg_elbow_hinge: axis 0 1 0 -> 0 0 1; child left_front_elbow_ball -> left_front_calf; limit lower=-.79 upper=.79 effort=1000 velocity=1 -> lower=-1.57 upper=1.57 effort=100 velocity=1; origin xyz=0 0 -1.9 rpy=0 0 0 -> xyz=0.4 0 0 rpy=0 0 0
- joint left_front_leg_shoulder_hinge: axis 1 0 0 -> 0 0 1; child left_front_leg -> left_front_shoulder; limit lower=-.52 upper=1.57 effort=1000 velocity=1 -> lower=-1.57 upper=1.57 effort=100 velocity=1; origin xyz=0 .125 0 rpy=0 0 0 -> xyz=0.5 .2 0 rpy=1.57 0 -1.57; parent left_front_shoulder -> base_link
- joint left_front_leg_shoulder_rotate: axis 0 1 0 -> 0 0 1; child left_front_shoulder -> left_front_leg; limit lower=-1.57 upper=1.57 effort=1000 velocity=1 -> lower=-1.57 upper=1.57 effort=100 velocity=1; origin xyz=1.5 .75 0 rpy=0 0 0 -> xyz=-.1 0 0 rpy=1.57 0 -1.57; parent base_link -> left_front_shoulder
- joint right_back_foot_hinge: origin xyz=0 0 -2 rpy=0 0 0 -> xyz=0.35 0 0 rpy=0 0 0
- joint right_back_leg_elbow_hinge: axis 0 1 0 -> 0 0 1; child right_back_elbow_ball -> right_back_calf; limit lower=-.79 upper=.79 effort=1000 velocity=1 -> lower=-1.57 upper=1.57 effort=100 velocity=1; origin xyz=0 0 -1.9 rpy=0 0 0 -> xyz=0.4 0 0 rpy=0 0 0
- joint right_back_leg_shoulder_hinge: axis 1 0 0 -> 0 0 1; child right_back_leg -> right_back_shoulder; limit lower=-.52 upper=1.57 effort=1000 velocity=1 -> lower=-1.57 upper=1.57 effort=100 velocity=1; origin xyz=0 -.125 0 rpy=0 0 0 -> xyz=-0.5 -.2 0 rpy=1.57 0 1.57; parent right_back_shoulder -> base_link
- joint right_back_leg_shoulder_rotate: axis 0 1 0 -> 0 0 1; child right_back_shoulder -> right_back_leg; limit lower=-1.57 upper=1.57 effort=1000 velocity=1 -> lower=-1.57 upper=1.57 effort=100 velocity=1; origin xyz=-1.5 -.75 0 rpy=0 0 0 -> xyz=-.1 0 0 rpy=1.57 0 -1.57; parent base_link -> right_back_shoulder
- joint right_front_foot_hinge: origin xyz=0 0 -2 rpy=0 0 0 -> xyz=0.35 0 0 rpy=0 0 0
- joint right_front_leg_elbow_hinge: axis 0 1 0 -> 0 0 1; child right_front_elbow_ball -> right_front_calf; limit lower=-.79 upper=.79 effort=1000 velocity=1 -> lower=-1.57 upper=1.57 effort=100 velocity=1; origin xyz=0 0 -1.9 rpy=0 0 0 -> xyz=0.4 0 0 rpy=0 0 0
- joint right_front_leg_shoulder_hinge: axis 1 0 0 -> 0 0 1; child right_front_leg -> right_front_shoulder; limit lower=-.52 upper=1.57 effort=1000 velocity=1 -> lower=-1.57 upper=1.57 effort=100 velocity=1; origin xyz=0 -.125 0 rpy=0 0 0 -> xyz=0.5 -.2 0 rpy=1.57 0 1.57; parent right_front_shoulder -> base_link
- joint right_front_leg_shoulder_rotate: axis 0 1 0 -> 0 0 1; child right_front_shoulder -> right_front_leg; limit lower=-1.57 upper=1.57 effort=1000 velocity=1 -> lower=-1.57 upper=1.57 effort=100 velocity=1; origin xyz=1.5 -.75 0 rpy=0 0 0 -> xyz=-.1 0 0 rpy=1.57 0 -1.57; parent base_link -> right_front_shoulder

Commit message: trabalho finalizado, continuar desenvolvimento

File: urdf/model2.urdf (robot description, URDF)
Before this commit: robot quadrupedal_robot, 18 links, 17 joints
Links:
- added link imu_link, mass 0
Joints:
- added joint imu_dummy: type fixed, parent base_link, child imu_link

Commit message: segunda parte concluída

File: urdf/model2.urdf (robot description, URDF)
Before this commit: robot quadrupedal_robot, 19 links, 18 joints
Links:
- removed link imu_link
- added link box_link, mass .5; collision box size=.25 .25 .25; visual box size=.25 .25 .25
- added link imu_cargo_link, mass 0
- added link imu_robot_link, mass 0
Joints:
- removed joint imu_dummy
- added joint imu_cargo_dummy: type fixed, parent box_link, child imu_cargo_link
- added joint imu_robot_dummy: type fixed, parent base_link, child imu_robot_link
- added joint spring: type prismatic, parent base_link, child box_link, origin xyz=0 0 .1 rpy=0 0 0, axis 0 0 1, limit lower=-.1 upper=.1 effort=1000 velocity=1000
- joint left_back_leg_elbow_hinge: limit lower=-1.57 upper=1.57 effort=100 velocity=1 -> lower=-1.57 upper=1.57 effort=100 velocity=100
- joint left_back_leg_shoulder_hinge: limit lower=-1.57 upper=1.57 effort=100 velocity=1 -> lower=-1.57 upper=1.57 effort=100 velocity=100
- joint left_back_leg_shoulder_rotate: limit lower=-1.57 upper=1.57 effort=100 velocity=1 -> lower=-1.57 upper=1.57 effort=100 velocity=100
- joint left_front_leg_elbow_hinge: limit lower=-1.57 upper=1.57 effort=100 velocity=1 -> lower=-1.57 upper=1.57 effort=100 velocity=100
- joint left_front_leg_shoulder_hinge: limit lower=-1.57 upper=1.57 effort=100 velocity=1 -> lower=-1.57 upper=1.57 effort=100 velocity=100
- joint left_front_leg_shoulder_rotate: limit lower=-1.57 upper=1.57 effort=100 velocity=1 -> lower=-1.57 upper=1.57 effort=100 velocity=100
- joint right_back_leg_elbow_hinge: limit lower=-1.57 upper=1.57 effort=100 velocity=1 -> lower=-1.57 upper=1.57 effort=100 velocity=100
- joint right_back_leg_shoulder_hinge: limit lower=-1.57 upper=1.57 effort=100 velocity=1 -> lower=-1.57 upper=1.57 effort=100 velocity=100
- joint right_back_leg_shoulder_rotate: limit lower=-1.57 upper=1.57 effort=100 velocity=1 -> lower=-1.57 upper=1.57 effort=100 velocity=100
- joint right_front_leg_elbow_hinge: limit lower=-1.57 upper=1.57 effort=100 velocity=1 -> lower=-1.57 upper=1.57 effort=100 velocity=100
- joint right_front_leg_shoulder_hinge: limit lower=-1.57 upper=1.57 effort=100 velocity=1 -> lower=-1.57 upper=1.57 effort=100 velocity=100
- joint right_front_leg_shoulder_rotate: limit lower=-1.57 upper=1.57 effort=100 velocity=1 -> lower=-1.57 upper=1.57 effort=100 velocity=100

Commit message: translating comments

File: urdf/model2.urdf (robot description, URDF)
Before this commit: robot quadrupedal_robot, 18 links, 17 joints
Links:
- link base_link: geometry collision box size=1 .4 .2; visual box size=1 .4 .2
Joints:
- joint left_back_leg_elbow_hinge: limit lower=-1.57 upper=1.57 effort=100 velocity=1 -> lower=-3.14159 upper=3.14159 effort=1000 velocity=10
- joint left_back_leg_shoulder_hinge: limit lower=-1.57 upper=1.57 effort=100 velocity=1 -> lower=-1.57 upper=1.57 effort=1000 velocity=10
- joint left_back_leg_shoulder_rotate: limit lower=-1.57 upper=1.57 effort=100 velocity=1 -> lower=-1.57 upper=1.57 effort=1000 velocity=10
- joint left_front_leg_elbow_hinge: limit lower=-1.57 upper=1.57 effort=100 velocity=1 -> lower=-3.14159 upper=3.14159 effort=1000 velocity=10
- joint left_front_leg_shoulder_hinge: limit lower=-1.57 upper=1.57 effort=100 velocity=1 -> lower=-1.57 upper=1.57 effort=1000 velocity=10
- joint left_front_leg_shoulder_rotate: limit lower=-1.57 upper=1.57 effort=100 velocity=1 -> lower=-1.57 upper=1.57 effort=1000 velocity=10
- joint right_back_leg_elbow_hinge: limit lower=-1.57 upper=1.57 effort=100 velocity=1 -> lower=-3.14159 upper=3.14159 effort=1000 velocity=10
- joint right_back_leg_shoulder_hinge: limit lower=-1.57 upper=1.57 effort=100 velocity=1 -> lower=-1.57 upper=1.57 effort=1000 velocity=10
- joint right_back_leg_shoulder_rotate: limit lower=-1.57 upper=1.57 effort=100 velocity=1 -> lower=-1.57 upper=1.57 effort=1000 velocity=10
- joint right_front_leg_elbow_hinge: limit lower=-1.57 upper=1.57 effort=100 velocity=1 -> lower=-3.14159 upper=3.14159 effort=1000 velocity=10
- joint right_front_leg_shoulder_hinge: limit lower=-1.57 upper=1.57 effort=100 velocity=1 -> lower=-1.57 upper=1.57 effort=1000 velocity=10
- joint right_front_leg_shoulder_rotate: limit lower=-1.57 upper=1.57 effort=100 velocity=1 -> lower=-1.57 upper=1.57 effort=1000 velocity=10
